File: keyboard.sch (KiCad schematic (older format))
At the start: 156 parts, among them J1 USB_C_Receptacle_USB2.0, K1 KEYSW, K10 KEYSW, K11 KEYSW, K12 KEYSW, K13 KEYSW, K14 KEYSW, K15 KEYSW, K16 KEYSW, K17 KEYSW, K18 KEYSW, K19 KEYSW, K2 KEYSW, K20 KEYSW, K21 KEYSW, K22 KEYSW, K23 KEYSW, K24 KEYSW, K25 KEYSW, K26 KEYSW, K27 KEYSW, K28 KEYSW, K29 KEYSW, K3 KEYSW, K30 KEYSW, K31 KEYSW, K32 KEYSW, K33 KEYSW, K34 KEYSW, K35 KEYSW, K36 KEYSW, K37 KEYSW, K38 KEYSW, K39 KEYSW, K4 KEYSW, K40 KEYSW, K41 KEYSW, K42 KEYSW, K43 KEYSW, K44 KEYSW, K45 KEYSW, K46 KEYSW, K47 KEYSW, K48 KEYSW, K49 KEYSW, K5 KEYSW, K50 KEYSW, K51 KEYSW, K52 KEYSW, K53 KEYSW, K54 KEYSW, K55 KEYSW, K56 KEYSW, K57 KEYSW, K58 KEYSW, K59 KEYSW, K6 KEYSW, K60 KEYSW, K61 KEYSW, K62 KEYSW, K63 KEYSW, K64 KEYSW, K65 KEYSW, K66 KEYSW, K67 KEYSW, K7 KEYSW, K8 KEYSW, K9 KEYSW, SW1 SW_PUSH, SW2 Rotary_Encoder_Switch, U1 ATMEGA32U4, X1 XTAL_GND

Commit message: updates
Parts:
- removed D54: D, symbol Device:D
- removed F1: 500mA, symbol Device:Polyfuse_Small
- removed K54: KEYSW, symbol keyboard_parts:KEYSW
- removed U1: ATMEGA32U4, symbol keyboard_parts:ATMEGA32U4
- removed X1: XTAL_GND, symbol keyboard_parts:XTAL_GND
- added U1: ATMEGA32U4-MU, ATMEGA32U4-MU:QFN50P700X700X100-45N, symbol ATMEGA32U4-MU:ATMEGA32U4-MU
- added Y1: Crystal_Small, Crystal:Crystal_SMD_3225-4Pin_3.2x2.5mm, symbol Device:Crystal_Small
- C1, C2, C3, C4, C5, C6, C7, C8: footprint Capacitor_SMD:C_0805_2012Metric_Pad1.18x1.45mm_HandSolder -> Capacitor_SMD:C_0603_1608Metric
- D1, D10, D11, D12, D13, D14, D15, D16, D17, D18, D19, D2, D20, D21, D22, D23, D24, D25, D26, D27, D28, D29, D3, D30, D31, D32, D33, D34, D35, D36, D37, D38, D39, D4, D40, D41, D42, D43, D5, D6, D7, D8, D9: footprint (none) -> Diode_SMD:D_0603_1608Metric
- D44: renamed from D45; footprint (none) -> Diode_SMD:D_0603_1608Metric
- D45: renamed from D46; footprint (none) -> Diode_SMD:D_0603_1608Metric
- D46: renamed from D47; footprint (none) -> Diode_SMD:D_0603_1608Metric
- D47: renamed from D48; footprint (none) -> Diode_SMD:D_0603_1608Metric
- D48: renamed from D49; footprint (none) -> Diode_SMD:D_0603_1608Metric
- D49: renamed from D50; footprint (none) -> Diode_SMD:D_0603_1608Metric
- D50: renamed from D51; footprint (none) -> Diode_SMD:D_0603_1608Metric
- D51: renamed from D52; footprint (none) -> Diode_SMD:D_0603_1608Metric
- D52: renamed from D53; footprint (none) -> Diode_SMD:D_0603_1608Metric
- D53: renamed from D44; footprint (none) -> Diode_SMD:D_0603_1608Metric
- D54: renamed from D55; footprint (none) -> Diode_SMD:D_0603_1608Metric
- D55: renamed from D56; footprint (none) -> Diode_SMD:D_0603_1608Metric
- D56: renamed from D57; footprint (none) -> Diode_SMD:D_0603_1608Metric
- D57: renamed from D58; footprint (none) -> Diode_SMD:D_0603_1608Metric
- D58: renamed from D59; footprint (none) -> Diode_SMD:D_0603_1608Metric
- D59: renamed from D60; footprint (none) -> Diode_SMD:D_0603_1608Metric
- D60: renamed from D61; footprint (none) -> Diode_SMD:D_0603_1608Metric
- D61: renamed from D62; footprint (none) -> Diode_SMD:D_0603_1608Metric
- D62: renamed from D63; footprint (none) -> Diode_SMD:D_0603_1608Metric
- D63: renamed from D64; footprint (none) -> Diode_SMD:D_0603_1608Metric
- D64: renamed from D65; footprint (none) -> Diode_SMD:D_0603_1608Metric
- D65: renamed from D66; footprint (none) -> Diode_SMD:D_0603_1608Metric
- D66: renamed from D67; footprint (none) -> Diode_SMD:D_0603_1608Metric
- D67: renamed from D68; footprint (none) -> Diode_SMD:D_0603_1608Metric
- J1: footprint (none) -> Connector_USB:USB_C_Receptacle_Amphenol_12401610E4-2A
- K1, K10, K11, K12, K13, K15, K16, K17, K18, K19, K20, K21, K22, K23, K24, K25, K26, K27, K28, K29, K30, K32, K33, K34, K35, K36, K37, K38, K39, K40, K41, K42, K43, K6, K7, K8: footprint (none) -> Button_Switch_Keyboard:SW_Cherry_MX_1.00u_PCB; symbol keyboard_parts:KEYSW -> keyboard-rescue:KEYSW-keyboard_parts
- K14, K5, K9: footprint (none) -> Button_Switch_Keyboard:SW_Cherry_MX_1.25u_PCB; symbol keyboard_parts:KEYSW -> keyboard-rescue:KEYSW-keyboard_parts
- K2: footprint (none) -> Button_Switch_Keyboard:SW_Cherry_MX_1.50u_PCB; symbol keyboard_parts:KEYSW -> keyboard-rescue:KEYSW-keyboard_parts
- K3: footprint (none) -> Button_Switch_Keyboard:SW_Cherry_MX_1.75u_PCB; symbol keyboard_parts:KEYSW -> keyboard-rescue:KEYSW-keyboard_parts
- K31: footprint (none) -> Button_Switch_Keyboard:SW_Cherry_MX_6.25u_PCB; symbol keyboard_parts:KEYSW -> keyboard-rescue:KEYSW-keyboard_parts
- K4: footprint (none) -> Button_Switch_Keyboard:SW_Cherry_MX_2.25u_PCB; symbol keyboard_parts:KEYSW -> keyboard-rescue:KEYSW-keyboard_parts
- K44: renamed from K45; footprint (none) -> Button_Switch_Keyboard:SW_Cherry_MX_1.00u_PCB; symbol keyboard_parts:KEYSW -> keyboard-rescue:KEYSW-keyboard_parts
- K45: renamed from K46; footprint (none) -> Button_Switch_Keyboard:SW_Cherry_MX_1.00u_PCB; symbol keyboard_parts:KEYSW -> keyboard-rescue:KEYSW-keyboard_parts
- K46: renamed from K47; footprint (none) -> Button_Switch_Keyboard:SW_Cherry_MX_1.00u_PCB; symbol keyboard_parts:KEYSW -> keyboard-rescue:KEYSW-keyboard_parts
- K47: renamed from K48; footprint (none) -> Button_Switch_Keyboard:SW_Cherry_MX_1.00u_PCB; symbol keyboard_parts:KEYSW -> keyboard-rescue:KEYSW-keyboard_parts
- K48: renamed from K49; footprint (none) -> Button_Switch_Keyboard:SW_Cherry_MX_1.25u_PCB; symbol keyboard_parts:KEYSW -> keyboard-rescue:KEYSW-keyboard_parts
- K49: renamed from K50; footprint (none) -> Button_Switch_Keyboard:SW_Cherry_MX_1.00u_PCB; symbol keyboard_parts:KEYSW -> keyboard-rescue:KEYSW-keyboard_parts
- K50: renamed from K51; footprint (none) -> Button_Switch_Keyboard:SW_Cherry_MX_1.00u_PCB; symbol keyboard_parts:KEYSW -> keyboard-rescue:KEYSW-keyboard_parts
- K51: renamed from K52; footprint (none) -> Button_Switch_Keyboard:SW_Cherry_MX_1.00u_PCB; symbol keyboard_parts:KEYSW -> keyboard-rescue:KEYSW-keyboard_parts
- K52: renamed from K53; footprint (none) -> Button_Switch_Keyboard:SW_Cherry_MX_1.00u_PCB; symbol keyboard_parts:KEYSW -> keyboard-rescue:KEYSW-keyboard_parts
- K53: renamed from K44; footprint (none) -> Button_Switch_Keyboard:SW_Cherry_MX_1.25u_PCB; symbol keyboard_parts:KEYSW -> keyboard-rescue:KEYSW-keyboard_parts
- K54: renamed from K55; footprint (none) -> Button_Switch_Keyboard:SW_Cherry_MX_1.00u_PCB; symbol keyboard_parts:KEYSW -> keyboard-rescue:KEYSW-keyboard_parts
- K55: renamed from K56; footprint (none) -> Button_Switch_Keyboard:SW_Cherry_MX_1.00u_PCB; symbol keyboard_parts:KEYSW -> keyboard-rescue:KEYSW-keyboard_parts
- K56: renamed from K57; footprint (none) -> Button_Switch_Keyboard:SW_Cherry_MX_1.75u_PCB; symbol keyboard_parts:KEYSW -> keyboard-rescue:KEYSW-keyboard_parts
- K57: renamed from K58; footprint (none) -> Button_Switch_Keyboard:SW_Cherry_MX_1.00u_PCB; symbol keyboard_parts:KEYSW -> keyboard-rescue:KEYSW-keyboard_parts
- K58: renamed from K59; footprint (none) -> Button_Switch_Keyboard:SW_Cherry_MX_2.00u_PCB; symbol keyboard_parts:KEYSW -> keyboard-rescue:KEYSW-keyboard_parts
- K59: renamed from K60; footprint (none) -> Button_Switch_Keyboard:SW_Cherry_MX_1.50u_PCB; symbol keyboard_parts:KEYSW -> keyboard-rescue:KEYSW-keyboard_parts
- K60: renamed from K61; footprint (none) -> Button_Switch_Keyboard:SW_Cherry_MX_2.25u_PCB; symbol keyboard_parts:KEYSW -> keyboard-rescue:KEYSW-keyboard_parts
- K61: renamed from K62; footprint (none) -> Button_Switch_Keyboard:SW_Cherry_MX_1.00u_PCB; symbol keyboard_parts:KEYSW -> keyboard-rescue:KEYSW-keyboard_parts
- K62: renamed from K63; footprint (none) -> Button_Switch_Keyboard:SW_Cherry_MX_1.00u_PCB; symbol keyboard_parts:KEYSW -> keyboard-rescue:KEYSW-keyboard_parts
- K63: renamed from K64; footprint (none) -> Button_Switch_Keyboard:SW_Cherry_MX_1.00u_PCB; symbol keyboard_parts:KEYSW -> keyboard-rescue:KEYSW-keyboard_parts
- K64: renamed from K65; footprint (none) -> Button_Switch_Keyboard:SW_Cherry_MX_1.00u_PCB; symbol keyboard_parts:KEYSW -> keyboard-rescue:KEYSW-keyboard_parts
- K65: renamed from K66; footprint (none) -> Button_Switch_Keyboard:SW_Cherry_MX_1.00u_PCB; symbol keyboard_parts:KEYSW -> keyboard-rescue:KEYSW-keyboard_parts
- K66: renamed from K67; footprint (none) -> Button_Switch_Keyboard:SW_Cherry_MX_1.00u_PCB; symbol keyboard_parts:KEYSW -> keyboard-rescue:KEYSW-keyboard_parts
- OLED1: footprint (none) -> oled:OLED-SSD1306
- R1: footprint (none) -> Resistor_SMD:R_0603_1608Metric; symbol Device:R -> Device:R_Small
- R2, R3, R4, R5, R6: footprint (none) -> Resistor_SMD:R_0603_1608Metric
- SW1: footprint (none) -> Button_Switch_THT:SW_PUSH_6mm; symbol keyboard_parts:SW_PUSH -> keyboard-rescue:SW_PUSH-keyboard_parts
- SW2: footprint (none) -> Rotary_Encoder:RotaryEncoder_Alps_EC11E-Switch_Vertical_H20mm
Connections:
- net D+: now also U1.4 (D+)
- net D-: now also U1.3 (D-)
- net VCC: now also J1.A4 (VBUS), J1.A9 (VBUS), J1.B4 (VBUS), J1.B9 (VBUS), U1.14 (VCC), U1.2 (UVCC), U1.24 (AVCC), U1.34 (VCC), U1.44 (AVCC), U1.7 (VBUS)
- net col11: now also K53.1
- net col9: no longer K53.1
- net hwb: now also U1.33 (PE2(~HWB~))
- net reset: now also U1.13 (~RESET~)
- net sck: now also U1.18 ((OC0B/SCL/INT0)PD0)
- net sda: now also U1.19 ((SDA/INT1)PD1)
- net ucap: now also U1.6 (UCAP)
- net xtal1: now also U1.17 (XTAL1), Y1.1
- net xtal2: now also U1.16 (XTAL2), Y1.2
- net +5V renamed GND
- net GND: now also U1.15 (GND), U1.23 (GND), U1.35 (GND), U1.43 (GND), U1.5 (UGND)
- no-connect marks 5 -> 3
Other:
- moved on the sheet: C1, C2, C3, C4, C5, C6, C7, C8, D53, J1, K53, OLED1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

Commit message: update
Parts:
- K1, K10, K11, K12, K13, K14, K15, K16, K17, K18, K19, K2, K20, K21, K22, K23, K24, K25, K26, K27, K28, K29, K3, K30, K31, K32, K33, K34, K35, K36, K37, K38, K39, K4, K40, K41, K42, K43, K44, K45, K46, K47, K48, K49, K5, K50, K51, K52, K53, K54, K55, K56, K57, K58, K59, K6, K60, K61, K62, K63, K64, K65, K66, K7, K8, K9: symbol keyboard-rescue:KEYSW-keyboard_parts -> Switch:SW_Push
- SW1: symbol keyboard-rescue:SW_PUSH-keyboard_parts -> Switch:SW_Push
Connections:
- net col0: now also K1.2, K2.2, K3.2, K4.2, K5.2; no longer K1.1, K2.1, K3.1, K4.1, K5.1
- net col1: now also K6.2, K7.2, K8.2, K9.2; no longer K6.1, K7.1, K8.1, K9.1
- net col10: now also K44.2, K45.2, K46.2, K47.2, K48.2; no longer K44.1, K45.1, K46.1, K47.1, K48.1
- net col11: now also K49.2, K50.2, K51.2, K52.2, K53.2; no longer K49.1, K50.1, K51.1, K52.1, K53.1
- net col12: now also K54.2, K55.2, K56.2, K57.2; no longer K54.1, K55.1, K56.1, K57.1
- net col13: now also K58.2, K59.2, K60.2, K61.2, K62.2; no longer K58.1, K59.1, K60.1, K61.1, K62.1
- net col14: now also K63.2, K64.2, K65.2, K66.2; no longer K63.1, K64.1, K65.1, K66.1
- net col2: now also K10.2, K11.2, K12.2, K13.2, K14.2; no longer K10.1, K11.1, K12.1, K13.1, K14.1
- net col3: now also K15.2, K16.2, K17.2, K18.2; no longer K15.1, K16.1, K17.1, K18.1
- net col4: now also K19.2, K20.2, K21.2, K22.2; no longer K19.1, K20.1, K21.1, K22.1
- net col5: now also K23.2, K24.2, K25.2, K26.2; no longer K23.1, K24.1, K25.1, K26.1
- net col6: now also K27.2, K28.2, K29.2, K30.2; no longer K27.1, K28.1, K29.1, K30.1, K31.1
- net col7: now also K32.2, K33.2, K34.2, K35.2; no longer K32.1, K33.1, K34.1, K35.1
- net col8: now also K36.2, K37.2, K38.2, K39.2; no longer K36.1, K37.1, K38.1, K39.1
- net col9: now also K40.2, K41.2, K42.2, K43.2; no longer K40.1, K41.1, K42.1, K43.1
- net at D54.2 (A): now also K54.1; no longer K54.2
- net at D58.2 (A): now also K58.1; no longer K58.2
- net at D11.2 (A): now also K11.1; no longer K11.2
- net at D12.2 (A): now also K12.1; no longer K12.2
- net at D13.2 (A): now also K13.1; no longer K13.2
- net at D14.2 (A): now also K14.1; no longer K14.2
- net at D16.2 (A): now also K16.1; no longer K16.2
- net at D17.2 (A): now also K17.1; no longer K17.2
- net at D18.2 (A): now also K18.1; no longer K18.2
- net at D20.2 (A): now also K20.1; no longer K20.2
- net at D21.2 (A): now also K21.1; no longer K21.2
- net at D22.2 (A): now also K22.1; no longer K22.2
- net at D24.2 (A): now also K24.1; no longer K24.2
- net at D28.2 (A): now also K28.1; no longer K28.2
- net at D33.2 (A): now also K33.1; no longer K33.2
- net at D37.2 (A): now also K37.1; no longer K37.2
- net at D41.2 (A): now also K41.1; no longer K41.2
- net at D45.2 (A): now also K45.1; no longer K45.2
- net at D25.2 (A): now also K25.1; no longer K25.2
- net at D29.2 (A): now also K29.1; no longer K29.2
- net at D34.2 (A): now also K34.1; no longer K34.2
- net at D38.2 (A): now also K38.1; no longer K38.2
- net at D42.2 (A): now also K42.1; no longer K42.2
- net at D46.2 (A): now also K46.1; no longer K46.2
- net at D10.2 (A): now also K10.1; no longer K10.2
- net at D15.2 (A): now also K15.1; no longer K15.2
- net at D1.2 (A): now also K1.1; no longer K1.2
- net at D19.2 (A): now also K19.1; no longer K19.2
- net at D23.2 (A): now also K23.1; no longer K23.2
- net at D27.2 (A): now also K27.1; no longer K27.2
- net at D32.2 (A): now also K32.1; no longer K32.2
- net at D36.2 (A): now also K36.1; no longer K36.2
- net at D40.2 (A): now also K40.1; no longer K40.2
- net at D44.2 (A): now also K44.1; no longer K44.2
- net at D26.2 (A): now also K26.1; no longer K26.2
- net at D30.2 (A): now also K30.1; no longer K30.2
- net at D35.2 (A): now also K35.1; no longer K35.2
- net at D39.2 (A): now also K39.1; no longer K39.2
- net at D43.2 (A): now also K43.1; no longer K43.2
- net at K31.2: no longer D31.2 (A)
- net at D2.2 (A): now also K2.1; no longer K2.2
- net at D3.2 (A): now also K3.1; no longer K3.2
- net at D4.2 (A): now also K4.1; no longer K4.2
- net at D50.2 (A): now also K50.1; no longer K50.2
- net at D55.2 (A): now also K55.1; no longer K55.2
- net at D59.2 (A): now also K59.1; no longer K59.2
- net at D63.2 (A): now also K63.1; no longer K63.2
- net at D51.2 (A): now also K51.1; no longer K51.2
- net at D60.2 (A): now also K60.1; no longer K60.2
- net at D64.2 (A): now also K64.1; no longer K64.2
- net at D5.2 (A): now also K5.1; no longer K5.2
- net at D49.2 (A): now also K49.1; no longer K49.2
- net at D6.2 (A): now also K6.1; no longer K6.2
- net at D7.2 (A): now also K7.1; no longer K7.2
- net at D8.2 (A): now also K8.1; no longer K8.2
- net at D47.2 (A): now also K47.1; no longer K47.2
- net at D52.2 (A): now also K52.1; no longer K52.2
- net at D61.2 (A): now also K61.1; no longer K61.2
- net at D65.2 (A): now also K65.1; no longer K65.2
- net at D48.2 (A): now also K48.1; no longer K48.2
- net at D57.2 (A): now also K57.1; no longer K57.2
- net at D62.2 (A): now also K62.1; no longer K62.2
- net at D66.2 (A): now also K66.1; no longer K66.2
- net at D9.2 (A): now also K9.1; no longer K9.2
- net at D56.2 (A): now also K56.1; no longer K56.2
- net at D53.2 (A): now also K53.1; no longer K53.2
Other:
- moved on the sheet: SW1

Commit message: position diodes
Connections:
- net GND: no longer C4.2, C5.2, C6.2, J1.A1 (GND), J1.A12 (GND), J1.B1 (GND), J1.B12 (GND), J1.S1 (SHIELD)
- net VCC: no longer C4.1, C5.1, C6.1
- net reset: no longer R1.1
- net row0: no longer D1.1 (K), D10.1 (K), D15.1 (K), D19.1 (K), D23.1 (K), D27.1 (K), D32.1 (K), D36.1 (K), D40.1 (K), D44.1 (K), D49.1 (K), D54.1 (K), D58.1 (K), D6.1 (K)
- net row1: no longer D11.1 (K), D16.1 (K), D2.1 (K), D20.1 (K), D24.1 (K), D28.1 (K), D33.1 (K), D37.1 (K), D41.1 (K), D45.1 (K), D50.1 (K), D55.1 (K), D59.1 (K), D7.1 (K)
- net row2: no longer D12.1 (K), D17.1 (K), D21.1 (K), D25.1 (K), D29.1 (K), D3.1 (K), D34.1 (K), D38.1 (K), D42.1 (K), D46.1 (K), D51.1 (K), D60.1 (K), D8.1 (K)
- net row3: no longer D13.1 (K), D18.1 (K), D22.1 (K), D26.1 (K), D30.1 (K), D35.1 (K), D39.1 (K), D4.1 (K), D43.1 (K), D47.1 (K), D52.1 (K), D56.1 (K), D61.1 (K)
- net row4: no longer D14.1 (K), D31.1 (K), D48.1 (K), D5.1 (K), D53.1 (K), D57.1 (K), D62.1 (K), D9.1 (K)
- net at J1.A6 (D+), J1.B6 (D+): no longer R6.2
- net at J1.A7 (D-), J1.B7 (D-): no longer R5.2
- new net: J1.A1 (GND), J1.A12 (GND), J1.B1 (GND), J1.B12 (GND), J1.S1 (SHIELD)

Commit message: routing
Parts:
- added K63: KEYSW, Button_Switch_Keyboard:SW_Cherry_MX_1.00u_PCB, symbol Switch:SW_Push
- renumbered D67 to D63, D63 to D64, D64 to D65, D65 to D66, D66 to D67, K63 to K64, K64 to K65, K65 to K66, K66 to K67
Connections:
- net GND: now also C4.2, C5.2, C6.2, J1.A1 (GND), J1.A12 (GND), J1.B1 (GND), J1.B12 (GND), J1.S1 (SHIELD)
- net VCC: now also C4.1, C5.1, C6.1
- net col0: now also U1.12 ((PCINT7/OC0A/OC1C/~RTS~)PB7)
- net col1: now also U1.41 (PF0(ADC0))
- net col10: now also U1.29 (PB5(PCINT5/OC1A/~OC4B~/ADC))
- net col11: now also U1.28 (PB4(PCINT4/ADC11))
- net col12: now also U1.27 (PD7(T0/OC4D/ADC10))
- net col13: now also U1.26 (PD6(T1/~OC4D~/ADC9))
- net col14: now also U1.25 (PD4(ICP1/ADC8)), K63.2
- net col2: now also U1.40 (PF1(ADC1))
- net col3: now also U1.39 (PF4(ADC4/TCK))
- net col4: now also U1.38 (PF5(ADC5/TMS))
- net col5: now also U1.37 (PF6(ADC6/TDO))
- net col6: now also K31.2, U1.36 (PF7(ADC7/TDI))
- net col7: now also U1.32 (PC7(ICP3/CLK0/OC4A))
- net col8: now also U1.31 (PC6(OC3A/~OC4A~))
- net col9: now also U1.30 (PB6(PCINT6/OC1B/OC4B/ADC))
- net encA: now also U1.21 ((TXD1/INT3)PD3)
- net encB: now also U1.22 ((XCK1/~CTS~)PD5)
- net reset: now also R1.1
- net row0: now also D1.1 (K), D10.1 (K), D15.1 (K), D19.1 (K), D23.1 (K), D27.1 (K), D32.1 (K), D36.1 (K), D40.1 (K), D44.1 (K), D49.1 (K), D54.1 (K), D58.1 (K), D6.1 (K), U1.1 ((INT6/AIN0)PE6)
- net row1: now also D11.1 (K), D16.1 (K), D2.1 (K), D20.1 (K), D24.1 (K), D28.1 (K), D33.1 (K), D37.1 (K), D41.1 (K), D45.1 (K), D50.1 (K), D55.1 (K), D59.1 (K), D7.1 (K), U1.8 ((SS/PCINT0)PB0)
- net row2: now also D12.1 (K), D17.1 (K), D21.1 (K), D25.1 (K), D29.1 (K), D3.1 (K), D34.1 (K), D38.1 (K), D42.1 (K), D46.1 (K), D51.1 (K), D60.1 (K), D8.1 (K), U1.9 ((PCINT1/SCLK)PB1)
- net row3: now also D13.1 (K), D18.1 (K), D22.1 (K), D26.1 (K), D30.1 (K), D35.1 (K), D39.1 (K), D4.1 (K), D43.1 (K), D47.1 (K), D52.1 (K), D56.1 (K), D61.1 (K), U1.10 ((PDI/PCINT2/MOSI)PB2)
- net row4: now also D14.1 (K), D31.1 (K), D48.1 (K), D5.1 (K), D53.1 (K), D57.1 (K), D62.1 (K), D9.1 (K), U1.11 ((PDO/PCINT3/MISO)PB3)
- net at J1.A6 (D+), J1.B6 (D+): now also R6.2
- net at J1.A7 (D-), J1.B7 (D-): now also R5.2
- net at K31.1: now also D31.2 (A)
- net at D63.2 (A): now also K63.1; no longer SW2.S2
- net rowE: now reaches U1.20 ((RXD1/INT2)PD2)
- net rowE: now also SW2.S2
Other:
- moved on the sheet: C1, C2, C3, C4, C5, C6, C7, C8, D1, D10, D11, D12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

Commit message: finished. :)
Parts:
- added D68: D, Diode_SMD:D_0603_1608Metric, symbol Device:D
Connections:
- net rowE: now also D68.1 (K); no longer SW2.S2
- new net: D68.2 (A), SW2.S2
Changed lines of the file:
@@
 Wire Wire Line
 	14350 1200 14700 1200
-Text GLabel 13750 1100 0    50   Input ~ 0
+Text GLabel 13450 1100 0    50   Input ~ 0
 rowE
 Wire Wire Line
@@
 Text GLabel 8000 7750 2    50   Input ~ 0
 rowE
+$Comp
+L Device:D D68
+U 1 1 60846CBB
+P 13600 1100
+F 0 "D68" H 13600 1200 50  0000 R CNN
+F 1 "D" H 13550 1300 50  0000 R CNN
+F 2 "Diode_SMD:D_0603_1608Metric" H 13600 1100 50  0001 C CNN
+F 3 "~" H 13600 1100 50  0001 C CNN
+	1    13600 1100
+	1    0    0    -1
+$EndComp
 $EndSCHEMATC

Commit message: finishing files
Parts:
- D1, D10, D11, D12, D13, D14, D15, D16, D17, D18, D19, D2, D20, D21, D22, D23, D24, D25, D26, D27, D28, D29, D3, D30, D31, D32, D33, D34, D35, D36, D37, D38, D39, D4, D40, D41, D42, D43, D44, D45, D46, D47, D48, D49, D5, D50, D51, D52, D53, D54, D55, D56, D57, D58, D59, D6, D60, D61, D62, D63, D64, D65, D66, D67, D68, D7, D8, D9: footprint Diode_SMD:D_0603_1608Metric -> Diode_SMD:D_SOD-323
