File: _autosave-keyboard.kicad_pcb (KiCad board)
At the start: 2 copper layers, 154 parts, among them J1 USB_C_Receptacle_USB2.0, K1 KEYSW, K10 KEYSW, K11 KEYSW, K12 KEYSW, K13 KEYSW, K14 KEYSW, K15 KEYSW, K16 KEYSW, K17 KEYSW, K18 KEYSW, K19 KEYSW, K2 KEYSW, K20 KEYSW, K21 KEYSW, K22 KEYSW, K23 KEYSW, K24 KEYSW, K25 KEYSW, K26 KEYSW, K27 KEYSW, K28 KEYSW, K29 KEYSW, K3 KEYSW, K30 KEYSW, K31 KEYSW, K32 KEYSW, K33 KEYSW, K34 KEYSW, K35 KEYSW, K36 KEYSW, K37 KEYSW, K38 KEYSW, K39 KEYSW, K4 KEYSW, K40 KEYSW, K41 KEYSW, K42 KEYSW, K43 KEYSW, K44 KEYSW, K45 KEYSW, K46 KEYSW, K47 KEYSW, K48 KEYSW, K49 KEYSW, K5 KEYSW, K50 KEYSW, K51 KEYSW, K52 KEYSW, K53 KEYSW, K54 KEYSW, K55 KEYSW, K56 KEYSW, K57 KEYSW, K58 KEYSW, K59 KEYSW, K6 KEYSW, K60 KEYSW, K61 KEYSW, K62 KEYSW, K63 KEYSW, K64 KEYSW, K65 KEYSW, K66 KEYSW, K7 KEYSW, K8 KEYSW, K9 KEYSW, SW1 SW_PUSH, SW2 Rotary_Encoder_Switch, U1 ATMEGA32U4, X1 XTAL_GND

Commit message: updates
Parts:
- moved U1 144.5 mm to (203.7, 37.1)
- moved OLED1 22.7 mm to (308.4, 36.6)
- moved SW2 19.3 mm to (366.5, 39.1), turned to 180 degrees
- moved J1 7.88 mm to (82.8, 38.4)
Connections:
- K54 pad 1: col11 -> col12
- OLED1 pad 1: (no net) -> sda
- OLED1 pad 2: (no net) -> sck
- OLED1 pad 3: (no net) -> VCC
- OLED1 pad 4: (no net) -> ugnd
