File: keyboard.kicad_pcb (KiCad board)
At the start: 2 copper layers, 154 parts, among them J1 USB_C_Receptacle_USB2.0, K1 KEYSW, K10 KEYSW, K11 KEYSW, K12 KEYSW, K13 KEYSW, K14 KEYSW, K15 KEYSW, K16 KEYSW, K17 KEYSW, K18 KEYSW, K19 KEYSW, K2 KEYSW, K20 KEYSW, K21 KEYSW, K22 KEYSW, K23 KEYSW, K24 KEYSW, K25 KEYSW, K26 KEYSW, K27 KEYSW, K28 KEYSW, K29 KEYSW, K3 KEYSW, K30 KEYSW, K31 KEYSW, K32 KEYSW, K33 KEYSW, K34 KEYSW, K35 KEYSW, K36 KEYSW, K37 KEYSW, K38 KEYSW, K39 KEYSW, K4 KEYSW, K40 KEYSW, K41 KEYSW, K42 KEYSW, K43 KEYSW, K44 KEYSW, K45 KEYSW, K46 KEYSW, K47 KEYSW, K48 KEYSW, K49 KEYSW, K5 KEYSW, K50 KEYSW, K51 KEYSW, K52 KEYSW, K53 KEYSW, K54 KEYSW, K55 KEYSW, K56 KEYSW, K57 KEYSW, K58 KEYSW, K59 KEYSW, K6 KEYSW, K60 KEYSW, K61 KEYSW, K62 KEYSW, K63 KEYSW, K64 KEYSW, K65 KEYSW, K66 KEYSW, K7 KEYSW, K8 KEYSW, K9 KEYSW, SW1 SW_PUSH, SW2 Rotary_Encoder_Switch, U1 ATMEGA32U4, X1 XTAL_GND

Commit message: update
Parts:
- removed the D54 at (92.1, 165.2)
- removed X1: XTAL_GND, Crystal:Crystal_SMD_3225-4Pin_3.2x2.5mm
- added Y1: Crystal_Small, Crystal:Crystal_SMD_3225-4Pin_3.2x2.5mm, F.Cu at (225.3, 25.4)
- R1, R2, R3, R4, R5, R6: footprint Resistor_SMD:R_0201_0603Metric -> Resistor_SMD:R_0603_1608Metric
- U1: value ATMEGA32U4 -> ATMEGA32U4-MU; footprint Keebio-Parts:ATMEGA32U4-AU -> ATMEGA32U4-MU:QFN50P700X700X100-45N
- moved U1 148.4 mm to (180.6, 33.8)
- moved OLED1 22.7 mm to (308.4, 36.6)
- moved SW2 19.3 mm to (366.5, 39.1), turned to 180 degrees
- moved J1 7.88 mm to (82.8, 38.4)
Connections:
- K1 pad 1: col0 -> Net-(D1-Pad2)
- K1 pad 2: Net-(D1-Pad2) -> col0
- K10 pad 1: col2 -> Net-(D10-Pad2)
- K10 pad 2: Net-(D10-Pad2) -> col2
- K11 pad 1: col2 -> Net-(D11-Pad2)
- K11 pad 2: Net-(D11-Pad2) -> col2
- K12 pad 1: col2 -> Net-(D12-Pad2)
- K12 pad 2: Net-(D12-Pad2) -> col2
- K13 pad 1: col2 -> Net-(D13-Pad2)
- K13 pad 2: Net-(D13-Pad2) -> col2
- K14 pad 1: col2 -> Net-(D14-Pad2)
- K14 pad 2: Net-(D14-Pad2) -> col2
- K15 pad 1: col3 -> Net-(D15-Pad2)
- K15 pad 2: Net-(D15-Pad2) -> col3
- K16 pad 1: col3 -> Net-(D16-Pad2)
- K16 pad 2: Net-(D16-Pad2) -> col3
- K17 pad 1: col3 -> Net-(D17-Pad2)
- K17 pad 2: Net-(D17-Pad2) -> col3
- K18 pad 1: col3 -> Net-(D18-Pad2)
- K18 pad 2: Net-(D18-Pad2) -> col3
- K19 pad 1: col4 -> Net-(D19-Pad2)
- K19 pad 2: Net-(D19-Pad2) -> col4
- K2 pad 1: col0 -> Net-(D2-Pad2)
- K2 pad 2: Net-(D2-Pad2) -> col0
- K20 pad 1: col4 -> Net-(D20-Pad2)
- K20 pad 2: Net-(D20-Pad2) -> col4
- K21 pad 1: col4 -> Net-(D21-Pad2)
- K21 pad 2: Net-(D21-Pad2) -> col4
- K22 pad 1: col4 -> Net-(D22-Pad2)
- K22 pad 2: Net-(D22-Pad2) -> col4
- K23 pad 1: col5 -> Net-(D23-Pad2)
- K23 pad 2: Net-(D23-Pad2) -> col5
- K24 pad 1: col5 -> Net-(D24-Pad2)
- K24 pad 2: Net-(D24-Pad2) -> col5
- K25 pad 1: col5 -> Net-(D25-Pad2)
- K25 pad 2: Net-(D25-Pad2) -> col5
- K26 pad 1: col5 -> Net-(D26-Pad2)
- K26 pad 2: Net-(D26-Pad2) -> col5
- K27 pad 1: col6 -> Net-(D27-Pad2)
- K27 pad 2: Net-(D27-Pad2) -> col6
- K28 pad 1: col6 -> Net-(D28-Pad2)
- K28 pad 2: Net-(D28-Pad2) -> col6
- K29 pad 1: col6 -> Net-(D29-Pad2)
- K29 pad 2: Net-(D29-Pad2) -> col6
- K3 pad 1: col0 -> Net-(D3-Pad2)
- K3 pad 2: Net-(D3-Pad2) -> col0
- K30 pad 1: col6 -> Net-(D30-Pad2)
- K30 pad 2: Net-(D30-Pad2) -> col6
- K31 pad 1: col6 -> Net-(K31-Pad1)
- K31 pad 2: Net-(D31-Pad2) -> Net-(K31-Pad2)
- K32 pad 1: col7 -> Net-(D32-Pad2)
- K32 pad 2: Net-(D32-Pad2) -> col7
- K33 pad 1: col7 -> Net-(D33-Pad2)
- K33 pad 2: Net-(D33-Pad2) -> col7
- K34 pad 1: col7 -> Net-(D34-Pad2)
- K34 pad 2: Net-(D34-Pad2) -> col7
- K35 pad 1: col7 -> Net-(D35-Pad2)
- K35 pad 2: Net-(D35-Pad2) -> col7
- K36 pad 1: col8 -> Net-(D36-Pad2)
- K36 pad 2: Net-(D36-Pad2) -> col8
- K37 pad 1: col8 -> Net-(D37-Pad2)
- K37 pad 2: Net-(D37-Pad2) -> col8
- K38 pad 1: col8 -> Net-(D38-Pad2)
- K38 pad 2: Net-(D38-Pad2) -> col8
- K39 pad 1: col8 -> Net-(D39-Pad2)
- K39 pad 2: Net-(D39-Pad2) -> col8
- K4 pad 1: col0 -> Net-(D4-Pad2)
- K4 pad 2: Net-(D4-Pad2) -> col0
- K40 pad 1: col9 -> Net-(D40-Pad2)
- K40 pad 2: Net-(D40-Pad2) -> col9
- K41 pad 1: col9 -> Net-(D41-Pad2)
- K41 pad 2: Net-(D41-Pad2) -> col9
- K42 pad 1: col9 -> Net-(D42-Pad2)
- K42 pad 2: Net-(D42-Pad2) -> col9
- K43 pad 1: col9 -> Net-(D43-Pad2)
- K43 pad 2: Net-(D43-Pad2) -> col9
- K44 pad 1: col10 -> Net-(D44-Pad2)
- K44 pad 2: Net-(D44-Pad2) -> col10
- K45 pad 1: col10 -> Net-(D45-Pad2)
- K45 pad 2: Net-(D45-Pad2) -> col10
- K46 pad 1: col10 -> Net-(D46-Pad2)
- K46 pad 2: Net-(D46-Pad2) -> col10
- K47 pad 1: col10 -> Net-(D47-Pad2)
- K47 pad 2: Net-(D47-Pad2) -> col10
- K48 pad 1: col10 -> Net-(D48-Pad2)
- K48 pad 2: Net-(D48-Pad2) -> col10
- K49 pad 1: col11 -> Net-(D49-Pad2)
- K49 pad 2: Net-(D49-Pad2) -> col11
- K5 pad 1: col0 -> Net-(D5-Pad2)
- K5 pad 2: Net-(D5-Pad2) -> col0
- K50 pad 1: col11 -> Net-(D50-Pad2)
- K50 pad 2: Net-(D50-Pad2) -> col11
- K51 pad 1: col11 -> Net-(D51-Pad2)
- K51 pad 2: Net-(D51-Pad2) -> col11
- K52 pad 1: col11 -> Net-(D52-Pad2)
- K52 pad 2: Net-(D52-Pad2) -> col11
- K53 pad 1: col11 -> Net-(D53-Pad2)
- K53 pad 2: Net-(D53-Pad2) -> col11
- K54 pad 1: col11 -> Net-(D54-Pad2)
- K54 pad 2: Net-(D54-Pad2) -> col12
- K55 pad 1: col12 -> Net-(D55-Pad2)
- K55 pad 2: Net-(D55-Pad2) -> col12
- K56 pad 1: col12 -> Net-(D56-Pad2)
- K56 pad 2: Net-(D56-Pad2) -> col12
- K57 pad 1: col12 -> Net-(D57-Pad2)
- K57 pad 2: Net-(D57-Pad2) -> col12
- K58 pad 1: col13 -> Net-(D58-Pad2)
- K58 pad 2: Net-(D58-Pad2) -> col13
- K59 pad 1: col13 -> Net-(D59-Pad2)
- K59 pad 2: Net-(D59-Pad2) -> col13
- K6 pad 1: col1 -> Net-(D6-Pad2)
- K6 pad 2: Net-(D6-Pad2) -> col1
- K60 pad 1: col13 -> Net-(D60-Pad2)
- K60 pad 2: Net-(D60-Pad2) -> col13
- K61 pad 1: col13 -> Net-(D61-Pad2)
- K61 pad 2: Net-(D61-Pad2) -> col13
- K62 pad 1: col13 -> Net-(D62-Pad2)
- K62 pad 2: Net-(D62-Pad2) -> col13
- K63 pad 1: col14 -> Net-(D63-Pad2)
- K63 pad 2: Net-(D63-Pad2) -> col14
- K64 pad 1: col14 -> Net-(D64-Pad2)
- K64 pad 2: Net-(D64-Pad2) -> col14
- K65 pad 1: col14 -> Net-(D65-Pad2)
- K65 pad 2: Net-(D65-Pad2) -> col14
- K66 pad 1: col14 -> Net-(D66-Pad2)
- K66 pad 2: Net-(D66-Pad2) -> col14
- K7 pad 1: col1 -> Net-(D7-Pad2)
- K7 pad 2: Net-(D7-Pad2) -> col1
- K8 pad 1: col1 -> Net-(D8-Pad2)
- K8 pad 2: Net-(D8-Pad2) -> col1
- K9 pad 1: col1 -> Net-(D9-Pad2)
- K9 pad 2: Net-(D9-Pad2) -> col1
- OLED1 pad 1: (no net) -> sda
- OLED1 pad 2: (no net) -> sck
- OLED1 pad 3: (no net) -> VCC
- OLED1 pad 4: (no net) -> ugnd
- U1 pad 16: xtal1 -> xtal2
- U1 pad 17: xtal2 -> xtal1

Commit message: position diodes
Parts:
- removed D67: D, Diode_SMD:D_0603_1608Metric
- C1, C2, C3, C4, C5, C6, C7, C8, D1, D10, D11, D12, D13, D14, D15, D16, D17, D18, D19, D2, D20, D21, D22, D23, D24, D25, D26, D27, D28, D29, D3, D30, D31, D32, D33, D34, D35, D36, D37, D38, D39, D4, D40, D41, D42, D43, D44, D45, D46, D47, D48, D49, D5, D50, D51, D52, D53, D54, D55, D56, D57, D58, D59, D6, D60, D61, D62, D63, D64, D65, D66, D7, D8, D9, R1, R2, R3, R4, R5, R6, SW1, U1, Y1: moved to B.Cu
- moved D63 292.5 mm to (365.4, 69.8), turned to 180 degrees
- moved D64 292.1 mm to (365.4, 88.8), turned to 180 degrees
- moved D65 291.5 mm to (365.4, 108.0), turned to 180 degrees
- moved D59 274.5 mm to (341.6, 69.8), turned to 180 degrees
- moved D58 274.3 mm to (336.8, 50.8), turned to 180 degrees
- moved D61 272.1 mm to (346.1, 108.0), turned to 180 degrees
- moved D66 268.0 mm to (365.4, 127.0), turned to 180 degrees
- moved D62 259.3 mm to (346.4, 127.0), turned to 180 degrees
- moved D54 243.3 mm to (308.2, 50.8), turned to 180 degrees
- moved D57 242.2 mm to (327.2, 127.0), turned to 180 degrees
- moved D55 238.2 mm to (317.8, 69.8), turned to 180 degrees
- moved D56 232.8 mm to (320.2, 108.0), turned to 180 degrees
- moved D46 202.2 mm to (284.4, 88.8), turned to 180 degrees
- moved D45 202.0 mm to (279.6, 69.8), turned to 180 degrees
- moved D44 198.7 mm to (270.2, 50.8), turned to 180 degrees
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
Commit message: routing
Parts:
- added D63: D, Diode_SMD:D_0603_1608Metric, B.Cu at (365.5, 50.8)
- added K63: KEYSW, Button_Switch_Keyboard:SW_Cherry_MX_1.00u_PCB, F.Cu at (361.9, 50.8)
- moved Y1 55.4 mm to (97.2, 37.1), turned to 225 degrees
- moved R5 48.6 mm to (77.0, 42.9), turned to 90 degrees
- moved R4 45.5 mm to (77.0, 38.9), turned to 270 degrees
- moved C8 44.8 mm to (68.3, 37.6), turned to 0 degrees
- moved R6 39.3 mm to (89.7, 42.9), turned to 90 degrees
- moved R3 30.5 mm to (89.7, 38.9), turned to 270 degrees
- moved C1 27.7 mm to (99.3, 34.8), turned to 135 degrees
- moved C2 22.7 mm to (95.0, 39.4), turned to 135 degrees
- moved OLED1 21.8 mm to (330.2, 37.2)
- moved R1 15.8 mm to (130.6, 35.3), turned to 90 degrees
- moved SW2 15.0 mm to (352.2, 34.8), turned to 0 degrees
- moved R2 11.2 mm to (110.2, 42.4)
- moved C5 9.59 mm to (116.3, 43.2), turned to 90 degrees
- moved C7 5.57 mm to (112.8, 43.2), turned to 90 degrees
- moved U1 5.36 mm to (102.9, 42.4), turned to 45 degrees
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- renumbered D63 to D64, D64 to D65, D65 to D66, D66 to D67, K63 to K64, K64 to K65, K65 to K66, K66 to K67
Connections:
- K31 pad 1: Net-(K31-Pad1) -> Net-(D31-Pad2)
- K31 pad 2: Net-(K31-Pad2) -> col6
- SW2 pad S2: Net-(D67-Pad2) (its old number) -> rowE
- U1 pad 1: Net-(U1-Pad1) -> row0
- U1 pad 10: Net-(U1-Pad10) -> row3
- U1 pad 11: Net-(U1-Pad11) -> row4
- U1 pad 12: Net-(U1-Pad12) -> col0
- U1 pad 20: Net-(U1-Pad20) -> rowE
- U1 pad 21: Net-(U1-Pad21) -> encA
- U1 pad 22: Net-(U1-Pad22) -> encB
- U1 pad 25: Net-(U1-Pad25) -> col14
- U1 pad 26: Net-(U1-Pad26) -> col13
- U1 pad 27: Net-(U1-Pad27) -> col12
- U1 pad 28: Net-(U1-Pad28) -> col11
- U1 pad 29: Net-(U1-Pad29) -> col10
- U1 pad 30: Net-(U1-Pad30) -> col9
- U1 pad 31: Net-(U1-Pad31) -> col8
- U1 pad 32: Net-(U1-Pad32) -> col7
- U1 pad 36: Net-(U1-Pad36) -> col6
- U1 pad 37: Net-(U1-Pad37) -> col5
- U1 pad 38: Net-(U1-Pad38) -> col4
- U1 pad 39: Net-(U1-Pad39) -> col3
- U1 pad 40: Net-(U1-Pad40) -> col2
- U1 pad 41: Net-(U1-Pad41) -> col1
- U1 pad 8: Net-(U1-Pad8) -> row1
- U1 pad 9: Net-(U1-Pad9) -> row2
Routing:
- net row4: track 0.00 -> 413.2 mm
- net row3: track 0.00 -> 393.3 mm
- net row2: track 0.00 -> 376.9 mm
- net row1: track 0.00 -> 359.2 mm
- net col14: track 0.00 -> 351.8 mm, vias 0 -> 1
- net col13: track 0.00 -> 317.2 mm, vias 0 -> 1
- net row0: track 0.00 -> 307.8 mm
- net col12: track 0.00 -> 286.2 mm, vias 0 -> 1
- net rowE: track 0.00 -> 280.1 mm
- net col11: track 0.00 -> 265.9 mm, vias 0 -> 1
- net encA: track 0.00 -> 260.4 mm
- net encB: track 0.00 -> 257.8 mm
- net col10: track 0.00 -> 250.1 mm, vias 0 -> 1
- net VCC: track 0.00 -> 242.6 mm, vias 0 -> 3
- net sda: track 0.00 -> 224.8 mm, vias 0 -> 1
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Other:
- board text added: "gryph"

Commit message: routing, drc
Parts:
- moved C8 29.8 mm to (96.7, 46.9), turned to 315 degrees
- moved C4 20.5 mm to (97.7, 45.8), turned to 135 degrees
- moved C5 16.5 mm to (100.6, 48.4), turned to 225 degrees
- moved R3 12.8 mm to (76.9, 40.6)
- moved R4 12.6 mm to (89.4, 40.6)
- moved C6 11.7 mm to (104.1, 48.3), turned to 225 degrees
- moved C7 10.5 mm to (104.9, 36.3), turned to 135 degrees
- moved C3 9.64 mm to (110.3, 43.6), turned to 0 degrees
- moved R6 8.07 mm to (81.6, 43.5), turned to 0 degrees
- moved R5 7.81 mm to (84.8, 43.5), turned to 180 degrees
- moved J1 2.39 mm to (83.2, 36.2)
- moved OLED1 2.10 mm to (330.9, 39.2)
- moved SW2 2.00 mm to (352.2, 36.7)
- moved R2 0.41 mm to (110.3, 42.0)
Routing:
- net col14: track 351.8 -> 557.9 mm
- net ugnd: track 32.4 -> 82.7 mm, vias 0 -> 1
- net reset: track 57.5 -> 102.0 mm, vias 0 -> 3
- net D+: track 0.00 -> 29.6 mm, vias 0 -> 2
- net D-: track 0.00 -> 23.3 mm, vias 0 -> 2
- net Net-(J1-PadB5): track 0.00 -> 12.0 mm
- net Net-(J1-PadA7): track 0.00 -> 8.85 mm, vias 0 -> 2
- net Net-(J1-PadA5): track 0.00 -> 6.32 mm
- net ucap: track 0.00 -> 4.67 mm
- net Net-(J1-PadA6): track 0.24 -> 4.28 mm
- net VCC: track 242.6 -> 245.7 mm, vias 3 -> 2
- net rowE: track 280.1 -> 281.5 mm
- net sck: track 223.1 -> 224.1 mm
- net sda: track 224.8 -> 225.7 mm
- net encB: track 257.8 -> 258.4 mm
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- added copper zone on B.Cu, net ugnd
- added copper zone on F.Cu, net ugnd
Other:
- board outline added: 304.8 x 109.3 mm
- board text added: "gryphon65"
- board text removed: "gryph"

Commit message: one more connection
Parts:
- moved C8 0.61 mm to (97.1, 47.3), turned to 0 degrees
- moved C4 0.60 mm to (97.1, 45.7), turned to 180 degrees
- moved C6 0.10 mm to (104.0, 48.4)
- moved C5 0.05 mm to (100.6, 48.4)
Routing:
- net VCC: track 245.7 -> 364.8 mm, vias 2 -> 9
- net reset: track 102.0 -> 60.1 mm, vias 3 -> 2
- net ugnd: track 82.7 -> 99.7 mm, vias 1 -> 8
- net col11: track 265.9 -> 269.4 mm
- net Net-(D13-Pad2): track 0.00 -> 2.77 mm
- net ucap: track 4.67 -> 3.63 mm
- net row0: track 307.8 -> 306.8 mm
- net col1: track 109.9 -> 110.7 mm
- net sda: track 225.7 -> 226.4 mm
Other:
- board text added: "gryphon67"
- board text removed: "gryphon65"

Commit message: finished. :)
Parts:
- added D68: D, Diode_SMD:D_0603_1608Metric, B.Cu at (363.8, 36.8)
Connections:
- SW2 pad S2: rowE -> Net-(D68-Pad2)
Routing:
- net rowE: track 281.6 -> 278.0 mm
- net VCC: track 364.8 -> 362.2 mm
- net ugnd: track 99.7 -> 102.2 mm
- net Net-(D68-Pad2): track 0.00 -> 2.06 mm
Other:
- board text added: "gryphon65"
- board text removed: "gryphon67"
